Commit message: Edit map inertia

File: urdf/maze.urdf (robot description, URDF)
Before this commit: robot map, 2 links, 1 joints
Links:
- link map: mass 0.836963110255319 -> 100

File: urdf/office.urdf (robot description, URDF)
Before this commit: robot map, 2 links, 1 joints
Links:
- link map: mass 0.836963110255319 -> 100
